File: output/pcbs/niu.kicad_pcb (KiCad board)
At the start: 2 copper layers, 244.8 x 127.3 mm, 106 parts

Commit message: Add mounting holes
Parts:
- moved S42 195.6 mm to (257.3, 145.2)
- moved S6 195.6 mm to (117.1, 140.8)
- moved S13 195.6 mm to (141.0, 100.3)
- moved D1 195.6 mm to (96.1, 157.0)
- moved S30 195.6 mm to (308.9, 95.9)
- moved S46 195.6 mm to (241.3, 172.3)
- moved S49 195.6 mm to (234.7, 115.7)
- moved S10 195.6 mm to (134.3, 156.9)
- moved D49 195.6 mm to (235.2, 120.1)
- moved S27 195.6 mm to (315.5, 152.5)
- moved D46 195.6 mm to (241.9, 176.7)
- moved S4 195.6 mm to (103.2, 95.9)
- moved S41 195.6 mm to (259.5, 164.1)
- moved D44 195.6 mm to (253.4, 112.0)
- moved D27 195.6 mm to (316.1, 157.0)
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Other:
- net class Default removed
