File: out/pcbs/keyboard-design.kicad_pcb (KiCad board)
At the start: 2 copper layers, 249.2 x 129.3 mm, 115 parts

Commit message: Finished mounting hole placement
Parts:
- added ?: , MountingHole_3.2mm_M3, F.Cu at (105.6, -64.6)
- added ?: , MountingHole_3.2mm_M3, F.Cu at (126.1, -64.6)
- added ?: , MountingHole_3.2mm_M3, F.Cu at (105.6, -41.6)
- added ?: , MountingHole_3.2mm_M3, F.Cu at (126.1, -41.6)
- moved MCU1 18.4 mm to (116.0, -88.0)
- moved OLED1 9.91 mm to (121.9, -66.7)
Changed lines of the file:
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@@
           )
       (module ProMicro (layer F.Cu)
-      (at 130 -100 270)
+      (at 116 -88 270)
       (fp_text reference "MCU1" (at 0 0) (layer F.SilkS) hide (effects (font (size 1.27 1.27) (thickness 0.15))))
       (fp_text value "" (at 0 0) (layer F.SilkS) hide (effects (font (size 1.27 1.27) (thickness 0.15))))
@@
     )
         (module lib:OLED_headers (layer F.Cu)
-        (at 115.884773 -74.5593585 270)
+        (at 121.87477299999999 -66.6593585 270)
         (fp_text reference "OLED1" (at 0 0) (layer F.SilkS) hide (effects (font (size 1.27 1.27) (thickness 0.15))))
         (fp_text value OLED (at 0 -7.3) (layer F.Fab) (effects (font (size 1 1) (thickness 0.15))))
@@
         )
 (module MountingHole_3.2mm_M3 (layer F.Cu)
+                    (at 105.634773 -64.5593585 0)
+		    (attr virtual)
+		    (descr "Mounting Hole 3.2mm, no annular, M3")
+		    (tags "mounting hole 3.2mm no annular m3")
+		    (fp_text user %R (at 0.3 0) (layer F.Fab)
+		     (effects (font (size 1 1) (thickness 0.15)))
+		    )
+		    (fp_circle (center 0 0) (end 3.2 0) (layer Cmts.User) (width 0.15))
+		    (fp_circle (center 0 0) (end 3.45 0) (layer F.CrtYd) (width 0.05))
+		    (pad 1 np_thru_hole circle (at 0 0) (size 3.2 3.2) (drill 3.2) (layers *.Cu *.Mask))
+		   )
+(module MountingHole_3.2mm_M3 (layer F.Cu)
+                    (at 126.134773 -64.5593585 0)
+		    (attr virtual)
+		    (descr "Mounting Hole 3.2mm, no annular, M3")
+		    (tags "mounting hole 3.2mm no annular m3")
+		    (fp_text user %R (at 0.3 0) (layer F.Fab)
+		     (effects (font (size 1 1) (thickness 0.15)))
+		    )
+		    (fp_circle (center 0 0) (end 3.2 0) (layer Cmts.User) (width 0.15))
+		    (fp_circle (center 0 0) (end 3.45 0) (layer F.CrtYd) (width 0.05))
+		    (pad 1 np_thru_hole circle (at 0 0) (size 3.2 3.2) (drill 3.2) (layers *.Cu *.Mask))
+		   )
+(module MountingHole_3.2mm_M3 (layer F.Cu)
+                    (at 105.634773 -41.5593585 0)
+		    (attr virtual)
+		    (descr "Mounting Hole 3.2mm, no annular, M3")
+		    (tags "mounting hole 3.2mm no annular m3")
+		    (fp_text user %R (at 0.3 0) (layer F.Fab)
+		     (effects (font (size 1 1) (thickness 0.15)))
+		    )
+		    (fp_circle (center 0 0) (end 3.2 0) (layer Cmts.User) (width 0.15))
+		    (fp_circle (center 0 0) (end 3.45 0) (layer F.CrtYd) (width 0.05))
+		    (pad 1 np_thru_hole circle (at 0 0) (size 3.2 3.2) (drill 3.2) (layers *.Cu *.Mask))
+		   )
+(module MountingHole_3.2mm_M3 (layer F.Cu)
+                    (at 126.134773 -41.5593585 0)
+		    (attr virtual)
+		    (descr "Mounting Hole 3.2mm, no annular, M3")
+		    (tags "mounting hole 3.2mm no annular m3")
+		    (fp_text user %R (at 0.3 0) (layer F.Fab)
+		     (effects (font (size 1 1) (thickness 0.15)))
+		    )
+		    (fp_circle (center 0 0) (end 3.2 0) (layer Cmts.User) (width 0.15))
+		    (fp_circle (center 0 0) (end 3.45 0) (layer F.CrtYd) (width 0.05))
+		    (pad 1 np_thru_hole circle (at 0 0) (size 3.2 3.2) (drill 3.2) (layers *.Cu *.Mask))
+		   )
+(module MountingHole_3.2mm_M3 (layer F.Cu)
                     (at 9.297879 -117.719155 -6.7)
